File: docs/e2e/2026-06-08-v2.4.0-release/screenshots/kicad/source/isolated_secondary.kicad_pcb (KiCad board)
At the start: 2 copper layers, 1315.6 x 354.8 mm, 21 parts

Commit message: Task 512: repair KiCad usability evidence
Parts:
- moved RBIAS1B 766.0 mm to (522.7, 19.1)
- moved RBIAS1A 728.0 mm to (500.8, 19.1)
- moved RPRE1B 690.0 mm to (478.9, 19.1)
- moved RPRE1A 652.0 mm to (457.0, 19.1)
- moved JSPK 614.0 mm to (405.8, 28.3)
- moved QOUT1 576.0 mm to (372.1, 44.3)
- moved QDRV1 538.0 mm to (344.8, 33.2)
- moved RVFILT1 500.0 mm to (319.0, 21.5)
- moved CFILT1 462.0 mm to (294.5, 18.4)
- moved RFILT1 424.0 mm to (272.9, 19.1)
- moved CTREBLE1 386.0 mm to (253.2, 18.4)
- moved RTREBLE1 348.1 mm to (231.6, 19.1)
- moved CMID1 310.1 mm to (211.9, 18.4)
- moved RMID1 272.1 mm to (190.3, 19.1)
- moved CBASS1 234.1 mm to (170.6, 18.4)
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Routing:
- net RBIAS1_INTERNAL_RBIAS1A_RBIAS1B: track 375.5 -> 37.6 mm
- net TONE1_INTERNAL_RTREBLE1_CTREBLE1: track 361.5 -> 36.1 mm
- net TONE1_INTERNAL_CMID1_RTREBLE1: track 347.6 -> 34.7 mm
- net TONE1_INTERNAL_RMID1_CMID1: track 333.5 -> 33.1 mm
- net TONE1_INTERNAL_CBASS1_RMID1: track 319.6 -> 31.7 mm
- net TONE1_INTERNAL_RBASS1_CBASS1: track 305.5 -> 30.1 mm
- net FILTER1_INTERNAL_CFILT1_RVFILT1: track 287.4 -> 52.4 mm
- net FILTER1_INTERNAL_RFILT1_CFILT1: track 277.5 -> 45.1 mm
- net RPRE1_INTERNAL_RPRE1A_RPRE1B: track 263.5 -> 43.6 mm
- net TONE_OUT: track 207.6 -> 37.7 mm
- net SPK_OUT: track 217.7 -> 63.7 mm
- net FILTER_OUT: track 226.1 -> 72.3 mm
- net PRE_OUT: track 192.3 -> 40.2 mm
- net DRV_OUT: track 198.8 -> 57.3 mm
- net GUITAR_IN: track 183.1 -> 66.1 mm
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Other:
- board size 1315.6 x 354.8 mm -> 543.6 x 96.8 mm
