File: docs/e2e/2026-06-08-v2.4.0-release/screenshots/kicad/source/isolated_secondary.kicad_sch (KiCad schematic)
At the start: 21 parts

Commit message: Task 512: repair KiCad usability evidence
Connections:
- net FILTER1_INTERNAL_CFILT1_RVFILT1 renamed N12
- net FILTER1_INTERNAL_RFILT1_CFILT1 renamed N11
- net RBIAS1_INTERNAL_RBIAS1A_RBIAS1B renamed N18
- net RPRE1_INTERNAL_RPRE1A_RPRE1B renamed N10
- net TONE1_INTERNAL_CBASS1_RMID1 renamed N14
- net TONE1_INTERNAL_CMID1_RTREBLE1 renamed N16
- net TONE1_INTERNAL_RBASS1_CBASS1 renamed N13
- net TONE1_INTERNAL_RMID1_CMID1 renamed N15
- net TONE1_INTERNAL_RTREBLE1_CTREBLE1 renamed N17
Other:
- note added: "MERLIN_NET: FILTER1_INTERNAL_CFILT1_RVFILT1"
- note added: "MERLIN_NET: FILTER1_INTERNAL_RFILT1_CFILT1"
- note added: "MERLIN_NET: NodeMap:FILTER1_INTERNAL_CFILT1_RVFILT1=N12"
- note added: "MERLIN_NET: NodeMap:FILTER1_INTERNAL_RFILT1_CFILT1=N11"
- note added: "MERLIN_NET: NodeMap:RBIAS1_INTERNAL_RBIAS1A_RBIAS1B=N18"
- note added: "MERLIN_NET: NodeMap:RPRE1_INTERNAL_RPRE1A_RPRE1B=N10"
- note added: "MERLIN_NET: NodeMap:TONE1_INTERNAL_CBASS1_RMID1=N14"
- note added: "MERLIN_NET: NodeMap:TONE1_INTERNAL_CMID1_RTREBLE1=N16"
- note added: "MERLIN_NET: NodeMap:TONE1_INTERNAL_RBASS1_CBASS1=N13"
- note added: "MERLIN_NET: NodeMap:TONE1_INTERNAL_RMID1_CMID1=N15"
- note added: "MERLIN_NET: NodeMap:TONE1_INTERNAL_RTREBLE1_CTREBLE1=N17"
- note added: "MERLIN_NET: RBIAS1_INTERNAL_RBIAS1A_RBIAS1B"
- note added: "MERLIN_NET: RPRE1_INTERNAL_RPRE1A_RPRE1B"
- note added: "MERLIN_NET: TONE1_INTERNAL_CBASS1_RMID1"
- note added: "MERLIN_NET: TONE1_INTERNAL_CMID1_RTREBLE1"
- note added: "MERLIN_NET: TONE1_INTERNAL_RBASS1_CBASS1"
- note added: "MERLIN_NET: TONE1_INTERNAL_RMID1_CMID1"
- note added: "MERLIN_NET: TONE1_INTERNAL_RTREBLE1_CTREBLE1"
- moved on the sheet: CBASS1, CFILT1, CMID1, CTREBLE1, JSPK, QDRV1, QOUT1, QPRE1, RBASS1, RBIAS1A, RBIAS1B, RFILT1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
